File: KiCadFiles/Castor.kicad_pcb (KiCad board)
At the start: 2 copper layers, 285.8 x 96.8 mm, 81 parts, among them J1 USB_C_Receptacle_USB2.0_14P, J2 USB_C_Receptacle_USB2.0_14P, J3 TRRS-L, J4 TRRS-R, SW1 SW_DPST_x2, SW2 SW_DPST_x2, SW3 SW_DPST_x2, SW4 SW_DPST_x2, U1 XC6206PxxxMR, U2 STM32F072CBTx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

Commit message: Add new DXF files for Castor project: introduced Castor-Edge_Cuts.dxf and Castor_border.dxf, while removing obsolete Edge_Cuts and User_2 DXF files. Updated PCB layout with new arc and line geometries, and refined UUIDs for edge cut elements. Adjusted plot path in project configuration for better file organization.
Other:
- board size 285.8 x 96.8 mm -> 293.8 x 105 mm

Commit message: Refactor KiCad project files for Castor: updated PCB layout with new component footprints and adjusted positions for resistors and capacitors. Removed obsolete audio jack symbol from schematic and added new power symbols for +3V3 and GND. Enhanced project configuration with updated track and via dimensions for improved design flexibility.
Parts:
- removed J3: TRRS-L, Connector_Audio:Jack_3.5mm_PJ320E_Horizontal
- removed J4: TRRS-R, Connector_Audio:Jack_3.5mm_PJ320E_Horizontal
- added J5: USB_C_Receptacle_USB2.0_14P, Connector_USB:USB_C_Receptacle_HRO_TYPE-C-31-M-12, F.Cu at (152.3, 67.9)
- added J6: USB_C_Receptacle_USB2.0_14P, Connector_USB:USB_C_Receptacle_HRO_TYPE-C-31-M-12, F.Cu at (164.4, 67.9)
- added R7: 5.1k, Resistor_SMD:R_0402_1005Metric, F.Cu at (168.2, 124.2)
- added R8: 5.1k, Resistor_SMD:R_0402_1005Metric, F.Cu at (168.2, 126.2)
- moved SW2 265.1 mm to (139.1, 75.5)
- moved SW1 265.0 mm to (139.3, 68.0)
- moved F1 247.3 mm to (144.7, 28.1)
- moved U3 233.3 mm to (150.9, 27.5)
- moved SW3 229.9 mm to (178.8, 67.1)
- moved SW4 229.8 mm to (178.8, 74.2)
- moved U1 228.1 mm to (151.3, 35.0)
- moved J1 222.4 mm to (139.3, 18.8), turned to 180 degrees
- moved U6 220.8 mm to (169.7, 27.4)
- moved C10 217.8 mm to (157.4, 126.3)
- moved C11 217.8 mm to (157.4, 128.2)
- moved C12 217.8 mm to (157.4, 130.2)
- moved C9 217.8 mm to (157.4, 124.3)
- moved C1 217.8 mm to (151.7, 124.3)
- moved C2 217.8 mm to (151.7, 126.3)
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Connections:
- MX1 pad 1: LEFT1 -> LEFT4
- MX10 pad 1: LEFT10 -> LEFT2
- MX11 pad 1: LEFT11 -> LEFT10
- MX12 pad 1: LEFT12 -> RIGHT30
- MX13 pad 1: LEFT13 -> RIGHT26
- MX14 pad 1: LEFT14 -> RIGHT27
- MX15 pad 1: LEFT15 -> LEFT9
- MX16 pad 1: LEFT16 -> LEFT11
- MX17 pad 1: LEFT17 -> LEFT12
- MX18 pad 1: LEFT18 -> RIGHT28
- MX19 pad 1: LEFT19 -> RIGHT29
- MX2 pad 1: LEFT2 -> RIGHT24
- MX20 pad 1: LEFT20 -> RIGHT31
- MX21 pad 1: LEFT21 -> LEFT7
- MX22 pad 1: RIGHT22 -> LEFT8
- MX23 pad 1: RIGHT23 -> LEFT16
- MX24 pad 1: RIGHT24 -> RIGHT36
- MX25 pad 1: RIGHT25 -> RIGHT32
- MX26 pad 1: RIGHT26 -> RIGHT33
- MX27 pad 1: RIGHT27 -> LEFT15
- MX28 pad 1: RIGHT28 -> LEFT17
- MX29 pad 1: RIGHT29 -> LEFT18
- MX30 pad 1: RIGHT30 -> RIGHT34
- MX31 pad 1: RIGHT31 -> RIGHT35
- MX32 pad 1: RIGHT32 -> RIGHT37
- MX33 pad 1: RIGHT33 -> LEFT13
- MX34 pad 1: RIGHT34 -> LEFT14
- MX35 pad 1: RIGHT35 -> RIGHT38
- MX36 pad 1: RIGHT36 -> RIGHT39
- MX37 pad 1: RIGHT37 -> LEFT19
- MX38 pad 1: RIGHT38 -> RIGHT42
- MX39 pad 1: RIGHT39 -> LEFT20
- MX4 pad 1: LEFT4 -> LEFT5
- MX40 pad 1: RIGHT40 -> RIGHT41
- MX41 pad 1: RIGHT41 -> LEFT21
- MX42 pad 1: RIGHT42 -> RIGHT40
- MX5 pad 1: LEFT5 -> LEFT6
- MX6 pad 1: LEFT6 -> RIGHT22
- MX7 pad 1: LEFT7 -> RIGHT23
- MX8 pad 1: LEFT8 -> RIGHT25
- MX9 pad 1: LEFT9 -> LEFT1
- U2 pad 38: unconnected-(U2-PA15-Pad38) -> HAND_L
- U4 pad 38: unconnected-(U4-PA15-Pad38) -> HAND_R
Other:
- outline, holes or cut-outs redrawn

Commit message: Update KiCad project files for Castor: added new global labels for RST and BOOT signals in the schematic, adjusted their positions, and removed obsolete labels. Updated PCB layout with new net connections and refined component placements for improved design clarity.
Parts:
- moved R5 111.2 mm to (178.9, 25.2), turned to -90 degrees
- moved R3 106.5 mm to (175.9, 25.2), turned to -90 degrees
- moved R2 101.4 mm to (140.8, 25.2), turned to -90 degrees
- moved C15 100.4 mm to (171.0, 28.4), turned to 90 degrees
- moved C16 100.0 mm to (166.7, 30.4), turned to 90 degrees
- moved C7 99.8 mm to (149.9, 28.6), turned to 90 degrees
- moved R1 99.7 mm to (137.8, 25.2), turned to -90 degrees
- moved C6 98.3 mm to (145.6, 28.4), turned to 90 degrees
- moved C4 89.8 mm to (136.3, 41.7), turned to 90 degrees
- moved C11 87.3 mm to (183.8, 45.0)
- moved R7 86.7 mm to (141.6, 41.7), turned to 90 degrees
- moved C10 86.3 mm to (174.3, 41.6), turned to 90 degrees
- moved R8 85.5 mm to (179.7, 41.5), turned to 90 degrees
- moved C5 81.9 mm to (132.8, 45.3), turned to 180 degrees
- moved C3 81.0 mm to (132.8, 49.5), turned to 180 degrees
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Connections:
- C14 pad 1: RST-1 -> RST-R
- C8 pad 1: RST-1 -> RST-L
- R4 pad 1: BOOT-1 -> BOOT-L
- R6 pad 1: BOOT-1 -> BOOT-R
- SW1 pad 1: RST-1 -> RST-L
- SW2 pad 1: BOOT-1 -> BOOT-L
- SW3 pad 1: RST-1 -> RST-R
- SW4 pad 1: BOOT-1 -> BOOT-R
- U4 pad 44: BOOT-1 -> BOOT-R
- U4 pad 7: RST-1 -> RST-R
Routing:
- net +3V3: track 0.00 -> 143.7 mm
- net DP: track 0.00 -> 70.6 mm
- net DN: track 0.00 -> 66.9 mm
- net GND: track 0.00 -> 55.0 mm
- net USART2_TX: track 0.00 -> 50.5 mm
- net USART2_RX: track 0.00 -> 46.9 mm, vias 0 -> 2
- net +5V: track 0.00 -> 23.9 mm, vias 0 -> 4
- net VBUS: track 0.00 -> 20.4 mm
- net BOOT-L: track 0.00 -> 7.60 mm
- net RST-R: track 0.00 -> 7.59 mm
- net BOOT-R: track 0.00 -> 7.54 mm
- net RST-L: track 0.00 -> 7.50 mm
- net Net-(J1-CC1): track 0.00 -> 2.06 mm
- net Net-(J2-CC1): track 0.00 -> 2.05 mm
- net Net-(J1-CC2): track 0.00 -> 2.04 mm
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