File: KiCadFiles/Castor.kicad_pcb (KiCad board)
At the start: 2 copper layers, 293.8 x 105 mm, 83 parts, among them J1 USB_C_Receptacle_USB2.0_14P, J2 USB_C_Receptacle_USB2.0_14P, J5 USB_C_Receptacle_USB2.0_14P, J6 USB_C_Receptacle_USB2.0_14P, SW1 SW_DPST_x2, SW2 SW_DPST_x2, SW3 SW_DPST_x2, SW4 SW_DPST_x2, U1 XC6206PxxxMR, U2 STM32F072CBTx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

Commit message: updated PCB layout by rearranging net connections and correcting net labels for improved clarity. Added new global labels for BOOT and RST signals in the schematic while removing obsolete labels. Enhanced design consistency across components and connections.
Connections:
- U2 pad 44: BOOT-1 -> BOOT-L
- U2 pad 7: RST-1 -> RST-L
Routing:
- net LEFT1: track 0.00 -> 125.4 mm
- net LEFT13: track 0.00 -> 120.1 mm
- net LEFT7: track 0.00 -> 118.4 mm
- net RIGHT27: track 0.00 -> 116.7 mm
- net RIGHT33: track 0.00 -> 116.3 mm
- net RIGHT39: track 0.00 -> 114.7 mm
- net LEFT2: track 0.00 -> 107.2 mm
- net LEFT14: track 0.00 -> 102.6 mm
- net LEFT8: track 0.00 -> 100.0 mm
- net RIGHT26: track 0.00 -> 99.0 mm
- net RIGHT32: track 0.00 -> 98.7 mm
- net RIGHT38: track 0.00 -> 97.1 mm
- net LEFT3: track 0.00 -> 77.2 mm
- net LEFT9: track 0.00 -> 72.9 mm
- net LEFT15: track 0.00 -> 72.5 mm
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
Commit message: Update KiCad project files for Castor: added new DRC exclusions in the project configuration, adjusted solder mask clearance, and refined global labels in the schematic for improved clarity. Updated PCB layout with corrected net connections and enhanced design consistency across components.
Parts:
- removed D1: 1N4148WS, Diode_SMD:D_SOD-323
- moved R7 1.89 mm to (142.0, 39.8)
- moved C5 1.47 mm to (133.0, 43.9)
- moved R8 1.15 mm to (180.7, 41.0), turned to 45 degrees
- moved C4 0.94 mm to (135.3, 41.9)
Connections:
- U2 pad 14: unconnected-(U2-PA4-Pad14) -> LEFT18
- U2 pad 15: unconnected-(U2-PA5-Pad15) -> LEFT17
- U2 pad 16: unconnected-(U2-PA6-Pad16) -> LEFT16
- U2 pad 17: unconnected-(U2-PA7-Pad17) -> LEFT15
- U2 pad 18: unconnected-(U2-PB0-Pad18) -> LEFT14
- U2 pad 19: unconnected-(U2-PB1-Pad19) -> LEFT13
- U2 pad 2: unconnected-(U2-PC13-Pad2) -> LEFT11
- U2 pad 20: unconnected-(U2-PB2-Pad20) -> LEFT19
- U2 pad 21: unconnected-(U2-PB10-Pad21) -> LEFT20
- U2 pad 22: unconnected-(U2-PB11-Pad22) -> LEFT21
- U2 pad 3: unconnected-(U2-PC14-Pad3) -> LEFT10
- U2 pad 39: unconnected-(U2-PB3-Pad39) -> LEFT6
- U2 pad 4: unconnected-(U2-PC15-Pad4) -> LEFT9
- U2 pad 40: unconnected-(U2-PB4-Pad40) -> LEFT5
- U2 pad 41: unconnected-(U2-PB5-Pad41) -> LEFT4
- U2 pad 42: unconnected-(U2-PB6-Pad42) -> LEFT3
- U2 pad 43: unconnected-(U2-PB7-Pad43) -> LEFT2
- U2 pad 45: unconnected-(U2-PB8-Pad45) -> LEFT1
- U2 pad 46: unconnected-(U2-PB9-Pad46) -> LEFT12
- U2 pad 5: unconnected-(U2-PF0-Pad5) -> LEFT8
- U2 pad 6: unconnected-(U2-PF1-Pad6) -> LEFT7
- U4 pad 14: unconnected-(U4-PA4-Pad14) -> RIGHT40
- U4 pad 15: unconnected-(U4-PA5-Pad15) -> RIGHT41
- U4 pad 16: unconnected-(U4-PA6-Pad16) -> RIGHT42
- U4 pad 17: unconnected-(U4-PA7-Pad17) -> RIGHT39
- U4 pad 18: unconnected-(U4-PB0-Pad18) -> RIGHT38
- U4 pad 19: unconnected-(U4-PB1-Pad19) -> RIGHT37
- U4 pad 20: unconnected-(U4-PB2-Pad20) -> RIGHT36
- U4 pad 21: unconnected-(U4-PB10-Pad21) -> RIGHT35
- U4 pad 22: unconnected-(U4-PB11-Pad22) -> RIGHT34
- U4 pad 26: unconnected-(U4-PB13-Pad26) -> RIGHT33
- U4 pad 27: unconnected-(U4-PB14-Pad27) -> RIGHT32
- U4 pad 28: unconnected-(U4-PB15-Pad28) -> RIGHT31
- U4 pad 29: unconnected-(U4-PA8-Pad29) -> RIGHT30
- U4 pad 30: unconnected-(U4-PA9-Pad30) -> RIGHT29
- U4 pad 31: unconnected-(U4-PA10-Pad31) -> RIGHT28
- U4 pad 37: unconnected-(U4-PA14-Pad37) -> RIGHT27
- U4 pad 39: unconnected-(U4-PB3-Pad39) -> RIGHT26
- U4 pad 40: unconnected-(U4-PB4-Pad40) -> RIGHT25
- U4 pad 41: unconnected-(U4-PB5-Pad41) -> RIGHT24
- U4 pad 42: unconnected-(U4-PB6-Pad42) -> RIGHT23
- U4 pad 43: unconnected-(U4-PB7-Pad43) -> RIGHT22
Routing:
- net RIGHT42: track 19.9 -> 76.2 mm
- net LEFT20: track 26.7 -> 69.1 mm, vias 0 -> 2
- net RIGHT41: track 15.9 -> 57.9 mm
- net LEFT19: track 46.5 -> 86.7 mm, vias 0 -> 2
- net LEFT13: track 120.1 -> 159.6 mm, vias 0 -> 2
- net LEFT14: track 102.6 -> 139.9 mm, vias 0 -> 2
- net RIGHT39: track 114.7 -> 151.8 mm
- net RIGHT40: track 20.5 -> 56.9 mm
- net RIGHT38: track 97.1 -> 132.0 mm
- net LEFT15: track 72.5 -> 107.2 mm, vias 0 -> 2
- net GNDREF: track 0.00 -> 34.0 mm
- net RIGHT37: track 68.0 -> 100.6 mm
- net LEFT16: track 53.3 -> 85.5 mm, vias 0 -> 2
- net LEFT21: track 32.1 -> 62.3 mm, vias 0 -> 2
- net RIGHT36: track 48.8 -> 79.0 mm
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- added copper zone on B.Cu, net GND
- added copper zone on F.Cu, net GND
Other:
- board text added: "B"
- board text added: "CastorKBD"
- board text added: "R"

Commit message: Update KiCad project files for Castor: modified PCB layout with new UUIDs for various elements, adjusted layer selection and plot parameters, and added a new user-defined rectangle layer. Updated project configuration to ignore certain silk clearance warnings for improved design flexibility.
Parts:
- moved C11 2.51 mm to (182.0, 43.3), turned to 90 degrees
- moved C3 1.40 mm to (133.4, 50.7), turned to -90 degrees
- moved C5 0.85 mm to (133.8, 43.8), turned to 90 degrees
Routing:
- net GND: track 59.9 -> 62.1 mm
- net +3V3: track 194.7 -> 196.2 mm
- net USART2_TX: track 51.5 -> 50.8 mm
Other:
- outline, holes or cut-outs redrawn
